Commit message: update

File: kani_description/robot/kani.urdf.xacro (robot description, xacro)
@@ -2,4 +2,4 @@
 <robot name="kani" xmlns:xacro="http://www.ros.org/wiki/xacro">
   <xacro:include filename="$(find kani_description)/urdf/base.urdf.xacro"/>
-  <xacro:base/>
+  <xacro:kani_base/>
 </robot>

File: kani_description/urdf/base.urdf.xacro (robot description, xacro)
@@ -2,5 +2,5 @@
 <robot xmlns:xacro="http://www.ros.org/wiki/xacro">
   <xacro:property name="pi" value="3.1415926535897931" />
-  <xacro:macro name="base">
+  <xacro:macro name="kani_base">
     <link name="base_footprint">
       <visual>
@@ -55,4 +55,3 @@
     </link>
   </xacro:macro>
-  <xacro:base/>
 </robot>
