Commit message: update relative position

File: kani_description/urdf/base.transmission.xacro (robot description, xacro)
@@ -7,9 +7,9 @@
       <type>transmission_interface/SimpleTransmission</type>
       <joint name="${joint_name}">
-        <hardwareInterface>VelocityJointInterface</hardwareInterface>
+        <hardwareInterface>hardware_interface/VelocityJointInterface</hardwareInterface>
       </joint>
       <actuator name="${joint_name}_wheel_motor">
         <mechanicalReduction>1</mechanicalReduction>
-        <hardwareInterface>VelocityJointInterface</hardwareInterface>
+        <hardwareInterface>hardware_interface/VelocityJointInterface</hardwareInterface>
       </actuator>
     </transmission>
@@ -19,9 +19,9 @@
       <type>transmission_interface/SimpleTransmission</type>
       <joint name="${joint_name}">
-        <hardwareInterface>PositionJointInterface</hardwareInterface>
+        <hardwareInterface>hardware_interface/PositionJointInterface</hardwareInterface>
       </joint>
       <actuator name="${joint_name}_steer_motor">
         <mechanicalReduction>1</mechanicalReduction>
-        <hardwareInterface>PositionJointInterface</hardwareInterface>
+        <hardwareInterface>hardware_interface/PositionJointInterface</hardwareInterface>
       </actuator>
     </transmission>

File: kani_description/urdf/base.urdf.xacro (robot description, xacro)
@@ -3,4 +3,7 @@
   <!-- <xacro:include filename="$(find kani_description)/urdf/base.transmission.xacro"/> -->
   <!-- <xacro:include filename="$(find kani_description)/urdf/base.gazebo.xacro" /> -->
+  <xacro:include filename="$(find kani_description)/urdf/sensors/rplidar_A1.urdf.xacro" />
+  <xacro:include filename="$(find kani_description)/urdf/sensors/_d435.urdf.xacro" />
+  <xacro:property name="base_height" value="0.06" />
   <xacro:macro name="kani_base">
     <link name="base_footprint">
@@ -13,5 +16,5 @@
     </link>
     <joint name="base_footprint_joint" type="fixed">
-      <origin xyz="0 0 0" rpy="0 0 0"/>
+      <origin xyz="0 0 ${base_height}" rpy="0 0 0"/>
       <child link="base_link" />
       <parent link="base_footprint"/>
@@ -20,5 +23,5 @@
       <inertial>
         <origin
-          xyz="0.0 0.0 0.06"
+          xyz="0 0 0"
           rpy="0 0 0"/>
         <mass
@@ -34,5 +37,5 @@
       <visual>
         <origin
-          xyz="-0.125 -0.1 0.05"
+          xyz="-0.125 -0.1 0"
           rpy="${pi/2} 0 ${pi/2}"/>
         <geometry>
@@ -58,5 +61,11 @@
     <!-- <xacro:rwheel />
     <xacro:lwheel /> -->
-    <!-- Hokuyo utm30lx-->
+    <!-- intel realsense d435 utm30lx-->
+    <sensor_d435 parent="base_link">
+      <origin xyz="0 0 -1" rpy="0 0 0"/>
+    </sensor_d435>
+    <sensor_a1 parent="base_link" name="laser">
+      <origin xyz="0 0 1" rpy="0 0 0"/>
+    </sensor_a1>
     <!-- <xacro:hokuyo_utm30lx name="hokuyo" parent="base_link"/> -->
     <!-- <xacro:hokuyo_utm30lx_back name="hokuyo_back" parent="base_link"/> -->
