Commit message: xacro urdf structure

File: kani_description/urdf/base.urdf.xacro (robot description, xacro)
@@ -1,4 +1,6 @@
 <?xml version="1.0"?>
 <robot xmlns:xacro="http://www.ros.org/wiki/xacro">
+  <!-- <xacro:include filename="$(find kani_description)/urdf/base.transmission.xacro"/> -->
+  <!-- <xacro:include filename="$(find kani_description)/urdf/base.gazebo.xacro" /> -->
   <xacro:property name="pi" value="3.1415926535897931" />
   <xacro:macro name="kani_base">
@@ -6,7 +8,7 @@
       <visual>
         <origin xyz="0 0 0" rpy="0 0 0"/>
-	<geometry>
-	  <box size="0.001 0.001 0.001"/>
-	</geometry>
+        <geometry>
+          <box size="0.001 0.001 0.001"/>
+        </geometry>
       </visual>
     </link>
@@ -19,39 +21,47 @@
       <inertial>
         <origin
-	  xyz="0.0 0.0 0.0"
-	  rpy="0 0 0"/>
-	<mass
-	  value="0.05"/>
-	<inertia
-	  ixx="0.2"
-	  ixy="0"
-	  ixz="0"
-	  iyy="0.2"
-	  iyz="0"
-	  izz="0.2"/>
-	</inertial>
-	<visual>
- 	  <origin
-            xyz="0 0 0"
-	    rpy="0 0 0"/>
-	  <geometry>
-	    <mesh
-		filename="package://kani_description/STL/base.stl"/>
-	  </geometry>
-	<!--<material>
-	</material>-->
-	</visual>
-	<collision>
- 	  <origin
-            xyz="0 0 0"
-	    rpy="0 0 0"/>
-	  <geometry>
-	    <mesh
-		filename="package://kani_description/STL/base.stl"/>
-	  </geometry>
-	  <material>
-	  </material>
-	</collision>
+          xyz="0.0 0.0 0.0"
+          rpy="0 0 0"/>
+        <mass
+          value="0.05"/>
+        <inertia
+          ixx="0.2"
+          ixy="0"
+          ixz="0"
+          iyy="0.2"
+          iyz="0"
+          izz="0.2"/>
+      </inertial>
+      <visual>
+        <origin
+          xyz="0 0 0"
+          rpy="${-pi / 2} 0 0"/>
+        <geometry>
+          <mesh
+            filename="package://kani_description/STL/base.stl"/>
+        </geometry>
+        <!-- <material>
+        </material> -->
+      </visual>
+      <collision>
+        <origin
+          xyz="0 0 0"
+          rpy="0 0 0"/>
+        <geometry>
+          <mesh
+            filename="package://kani_description/STL/base.stl"/>
+        </geometry>
+        <!-- <material>
+        </material> -->
+      </collision>
     </link>
+    <!-- Wheel macros -->
+    <!-- <xacro:rwheel />
+    <xacro:lwheel /> -->
+    <!-- Hokuyo utm30lx-->
+    <!-- <xacro:hokuyo_utm30lx name="hokuyo" parent="base_link"/> -->
+    <!-- <xacro:hokuyo_utm30lx_back name="hokuyo_back" parent="base_link"/> -->
+    <!-- Extensions -->
+    <!-- <xacro:kani_base_gazebo/> -->
   </xacro:macro>
 </robot>

File: kani_description/urdf/test.urdf (robot description, URDF)
Before this commit: robot 4WDSR, 5 links, 4 joints
Links:
- link base: geometry visual cylinder length=0.6 radius=0.2
- link wheel-lb: geometry visual cylinder length=0.6 radius=0.2
- link wheel-lf: geometry visual cylinder length=0.6 radius=0.2
- link wheel-rb: geometry visual cylinder length=0.6 radius=0.2
- link wheel-rf: geometry visual cylinder length=0.6 radius=0.2

Commit message: fix inertia

File: kani_description/urdf/base.urdf.xacro (robot description, xacro)
@@ -27,5 +27,5 @@
           rpy="0 0 0"/>
         <mass
-          value="2"/>
+          value="5"/>
         <inertia
           ixx="4e-3"

File: kani_description/urdf/wheels.urdf.xacro (robot description, xacro)
@@ -15,12 +15,12 @@
           rpy="${pi/2} 0 0" /><!--0.00222524026865972 0.173009757872407 -0.000157420245397055-->
         <mass
-          value="0.1" />
-        <inertia
-          ixx="1e-5"
+          value="0.029" />
+        <inertia
+          ixx="0.0000114"
           ixy="0.0"
           ixz="0.0"
-          iyy="1e-5"
+          iyy="0.0000114"
           iyz="0.0"
-          izz="1e-5" />
+          izz="0.0000212" />
       </inertial>
       <visual>
@@ -70,12 +70,12 @@
           rpy="0 0 ${pi}" /><!--0.00222524026865972 0.173009757872407 -0.000157420245397055-->
         <mass
-          value="0.1" />
-        <inertia
-          ixx="6e-4"
-          ixy="0.0"
-          ixz="0.0"
-          iyy="6e-4"
-          iyz="0.0"
-          izz="6e-4" />
+          value="0.104" />
+        <inertia
+          ixx="0.0000447"
+          ixy="0.00"
+          ixz="0.00"
+          iyy="0.0000362"
+          iyz="0.00"
+          izz="0.0000303" />
       </inertial>
       <visual>
@@ -131,12 +131,12 @@
           rpy="${pi/2} 0 0" /><!--0.00222524026865972 0.173009757872407 -0.000157420245397055-->
         <mass
-          value="0.1" />
-        <inertia
-          ixx="1e-5"
+          value="0.029" />
+        <inertia
+          ixx="0.0000114"
           ixy="0.0"
           ixz="0.0"
-          iyy="1e-5"
+          iyy="0.0000114"
           iyz="0.0"
-          izz="1e-5" />
+          izz="0.0000212" />
       </inertial>
       <visual>
@@ -186,12 +186,12 @@
           rpy="0 0 ${pi}" /><!--0.00222524026865972 0.173009757872407 -0.000157420245397055-->
         <mass
-          value="0.1" />
-        <inertia
-          ixx="6e-4"
-          ixy="0.0"
-          ixz="0.0"
-          iyy="6e-4"
-          iyz="0.0"
-          izz="6e-4"/>
+          value="0.104" />
+        <inertia
+          ixx="0.0000447"
+          ixy="0.00"
+          ixz="0.00"
+          iyy="0.0000362"
+          iyz="0.00"
+          izz="0.0000303"/>
       </inertial>
       <visual>
@@ -247,12 +247,12 @@
           rpy="${-pi/2} 0 0"  /><!--0.00222524026865972 0.173009757872407 -0.000157420245397055-->
         <mass
-          value="0.1" />
-        <inertia
-          ixx="1e-5"
+          value="0.029" />
+        <inertia
+          ixx="0.0000114"
           ixy="0.0"
           ixz="0.0"
-          iyy="1e-5"
+          iyy="0.0000114"
           iyz="0.0"
-          izz="1e-5" />
+          izz="0.0000212" />
       </inertial>
       <visual>
@@ -302,12 +302,12 @@
           rpy="0 0 0"/><!--0.00222524026865972 0.173009757872407 -0.000157420245397055-->
         <mass
-          value="0.1" />
-        <inertia
-          ixx="6e-4"
-          ixy="0.0"
-          ixz="0.0"
-          iyy="6e-4"
-          iyz="0.0"
-          izz="6e-4"/>
+          value="0.104" />
+        <inertia
+          ixx="0.0000447"
+          ixy="0.00"
+          ixz="0.00"
+          iyy="0.0000362"
+          iyz="0.00"
+          izz="0.0000303"/>
       </inertial>
       <visual>
@@ -363,12 +363,12 @@
           rpy="${-pi/2} 0 0" /><!--0.00222524026865972 0.173009757872407 -0.000157420245397055-->
         <mass
-          value="0.1" />
-        <inertia
-          ixx="1e-5"
+          value="0.029" />
+        <inertia
+          ixx="0.0000114"
           ixy="0.0"
           ixz="0.0"
-          iyy="1e-5"
+          iyy="0.0000114"
           iyz="0.0"
-          izz="1e-5" />
+          izz="0.0000212" />
       </inertial>
       <visual>
@@ -418,12 +418,12 @@
           rpy="0 0 0" /><!--0.00222524026865972 0.173009757872407 -0.000157420245397055-->
         <mass
-          value="0.1" />
-        <inertia
-          ixx="6e-4"
-          ixy="0.0"
-          ixz="0.0"
-          iyy="6e-4"
-          iyz="0.0"
-          izz="6e-4"/>
+          value="0.104" />
+        <inertia
+          ixx="0.0000447"
+          ixy="0.00"
+          ixz="0.00"
+          iyy="0.0000362"
+          iyz="0.00"
+          izz="0.0000303"/>
       </inertial>
       <visual>

Commit message: fix frames

File: kani_description/urdf/base.urdf.xacro (robot description, xacro)
@@ -64,5 +64,5 @@
     </sensor_d435>
     <sensor_a1 parent="base_link" name="laser">
-      <origin xyz="0.02 0.03 0.02" rpy="0 0 0"/>
+      <origin xyz="0.02 0.03 0.02" rpy="0 0 ${-pi/2}"/>
     </sensor_a1>
     <!-- Extensions -->

File: kani_description/urdf/sensors/rplidar_A1.urdf.xacro (robot description, xacro)
@@ -14,5 +14,5 @@
     <link name="${name}_link">
       <visual>
-      <origin xyz=" -0.00714 0.00714 0" rpy="0 0 ${-pi/2}"/>
+      <origin xyz=" -0.00714 0.00714 0" rpy="0 0 0"/>
       <!-- -0.00714 0.00714 0 -->
         <geometry>
@@ -22,5 +22,5 @@
       </visual>
       <collision>
-        <origin xyz="-0.00714 0.00714 0" rpy="0 0 ${-pi/2}"/>
+        <origin xyz="-0.00714 0.00714 0" rpy="0 0 0"/>
         <geometry>
           <mesh filename="package://kani_description/meshes/rplidar.stl"/>
