Commit message: model 1.0

File: kani_description/robots/kani.urdf.xacro (robot description, xacro)
@@ -1,9 +1,15 @@
 <?xml version="1.0"?>
 <robot name="kani" xmlns:xacro="http://www.ros.org/wiki/xacro">
+  <xacro:property name="pi" value="3.1415926535897931" />
   <xacro:include filename="$(find kani_description)/urdf/base.urdf.xacro"/>
   <xacro:include filename="$(find kani_description)/urdf/wheels.urdf.xacro"/>
   <xacro:kani_base/>
-  <xacro:wheel parent="base_link" x="0" y="0" z="0" wheel_name="rightFront"/>
-  <xacro:wheel parent="base_link" x="10" y="10" z="0" wheel_name="leftFront"/>
-  <xacro:steer parent="base_link" x="10" y="10" z="0" steer_name="rightFront">
+  <xacro:rf_steer parent="base_link" x="0.092" y="-0.088" z="0" />
+  <xacro:lf_steer parent="base_link" x="0.092" y="0.088" z="0" />
+  <xacro:rb_steer parent="base_link" x="-0.092" y="-0.088" z="0"/>
+  <xacro:lb_steer parent="base_link" x="-0.092" y="0.088" z="0" />
+  <xacro:rf_wheel parent="rightFront_steer_link" x="0" y="0" z="0"/>
+  <xacro:lf_wheel parent="leftFront_steer_link" x="0" y="0" z="0" />
+  <xacro:rb_wheel parent="rightBack_steer_link" x="0" y="0" z="0" />
+  <xacro:lb_wheel parent="leftBack_steer_link" x="0" y="0" z="0" />
 </robot>

File: kani_description/robots/robot.urdf (robot description, URDF)
Before this commit: robot kani, 4 links, 3 joints
Links:
- removed link leftFront_link
- removed link rightFront_link
- added link leftBack_steer_link, mass 0.0963917377366023; collision mesh filename=package://kani_description/meshes/steer2.stl; visual mesh filename=package://kani_description/meshes/steer2.stl
- added link leftBack_wheel_link, mass 0.0963917377366023; collision mesh filename=package://kani_description/meshes/wheel.stl; visual mesh filename=package://kani_description/meshes/wheel.stl
- added link leftFront_steer_link, mass 0.0963917377366023; collision mesh filename=package://kani_description/meshes/steer2_m.stl; visual mesh filename=package://kani_description/meshes/steer2_m.stl
- added link leftFront_wheel_link, mass 0.0963917377366023; collision mesh filename=package://kani_description/meshes/wheel.stl; visual mesh filename=package://kani_description/meshes/wheel.stl
- added link rightBack_steer_link, mass 0.0963917377366023; collision mesh filename=package://kani_description/meshes/steer2_m.stl; visual mesh filename=package://kani_description/meshes/steer2_m.stl
- added link rightBack_wheel_link, mass 0.0963917377366023; collision mesh filename=package://kani_description/meshes/wheel.stl; visual mesh filename=package://kani_description/meshes/wheel.stl
- added link rightFront_steer_link, mass 0.0963917377366023; collision mesh filename=package://kani_description/meshes/steer2.stl; visual mesh filename=package://kani_description/meshes/steer2.stl
- added link rightFront_wheel_link, mass 0.0963917377366023; collision mesh filename=package://kani_description/meshes/wheel.stl; visual mesh filename=package://kani_description/meshes/wheel.stl
- link base_link: geometry collision mesh filename=package://kani_description/meshes/base.stl; visual mesh filename=package://kani_description/meshes/base.stl
Joints:
- removed joint leftFront_joint
- removed joint rightFront_joint
- added joint leftBack_steer_joint: type revolute, parent base_link, child leftBack_steer_link, origin xyz=-0.092 0.088 0 rpy=0 0 0, axis 0 0 1, limit lower=-1.57079632679 upper=1.57079632679 effort=500 velocity=500
- added joint leftBack_wheel_joint: type continuous, parent leftBack_steer_link, child leftBack_wheel_link, origin xyz=0 0 0 rpy=0 0 0, axis 0 1 0
- added joint leftFront_steer_joint: type revolute, parent base_link, child leftFront_steer_link, origin xyz=0.092 0.088 0 rpy=0 0 0, axis 0 0 1, limit lower=-1.57079632679 upper=1.57079632679 effort=500 velocity=500
- added joint leftFront_wheel_joint: type continuous, parent leftFront_steer_link, child leftFront_wheel_link, origin xyz=0 0 0.005 rpy=0 0 0, axis 0 1 0
- added joint rightBack_steer_joint: type revolute, parent base_link, child rightBack_steer_link, origin xyz=-0.092 -0.088 0 rpy=0 0 0, axis 0 0 1, limit lower=-1.57079632679 upper=1.57079632679 effort=500 velocity=500
- added joint rightBack_wheel_joint: type continuous, parent rightBack_steer_link, child rightBack_wheel_link, origin xyz=0 0 0.015 rpy=0 0 0, axis 0 1 0
- added joint rightFront_steer_joint: type revolute, parent base_link, child rightFront_steer_link, origin xyz=0.092 -0.088 0 rpy=0 0 0, axis 0 0 1, limit lower=-1.57079632679 upper=1.57079632679 effort=500 velocity=500
- added joint rightFront_wheel_joint: type continuous, parent rightFront_steer_link, child rightFront_wheel_link, origin xyz=0 0 0.01 rpy=0 0 0, axis 0 1 0

File: kani_description/urdf/base.gazebo.xacro (robot description, xacro)
@@ -27,5 +27,5 @@
     <gazebo reference="${link_name}">
       <material>Gazebo/Red</material>
-      <!-- fix below params -->
+      <!-- fix below params?-->
       <mu1 value="100.0"/>
       <mu2 value="100.0"/>
@@ -34,5 +34,5 @@
       <fdir1 value="1 0 0"/>
       <dampingFactor value="0.1"/>
-      <!-- fix above params -->
+      <!-- fix above params? -->
     </gazebo>
   </xacro:macro>

File: kani_description/urdf/base.transmission.xacro (robot description, xacro)
@@ -4,10 +4,10 @@
   <!-- wheel transmission -->
   <xacro:macro name="kani_wheel_trans" params="joint_name">
-    <transmission name="${wheel_name}" type="SimpleTransmission">
+    <transmission name="${joint_name}_trans" type="SimpleTransmission">
       <type>transmission_interface/SimpleTransmission</type>
       <joint name="${joint_name}">
         <hardwareInterface>VelocityJointInterface</hardwareInterface>
       </joint>
-      <actuator name="${wheel_name}_wheel_motor">
+      <actuator name="${joint_name}_wheel_motor">
         <mechanicalReduction>1</mechanicalReduction>
         <hardwareInterface>VelocityJointInterface</hardwareInterface>
@@ -16,10 +16,10 @@
   </xacro:macro>
   <xacro:macro name="kani_steer_trans" params="joint_name">
-    <transmission name="${steer_name}" type="SimpleTransmission">
+    <transmission name="${joint_name}_trans" type="SimpleTransmission">
       <type>transmission_interface/SimpleTransmission</type>
       <joint name="${joint_name}">
         <hardwareInterface>PositionJointInterface</hardwareInterface>
       </joint>
-      <actuator name="${steer_name}_steer_motor">
+      <actuator name="${joint_name}_steer_motor">
         <mechanicalReduction>1</mechanicalReduction>
         <hardwareInterface>PositionJointInterface</hardwareInterface>

File: kani_description/urdf/base.urdf.xacro (robot description, xacro)
@@ -3,5 +3,4 @@
   <!-- <xacro:include filename="$(find kani_description)/urdf/base.transmission.xacro"/> -->
   <!-- <xacro:include filename="$(find kani_description)/urdf/base.gazebo.xacro" /> -->
-  <xacro:property name="pi" value="3.1415926535897931" />
   <xacro:macro name="kani_base">
     <link name="base_footprint">
@@ -21,5 +20,5 @@
       <inertial>
         <origin
-          xyz="0.0 0.0 0.0"
+          xyz="0.0 0.0 0.06"
           rpy="0 0 0"/>
         <mass
@@ -35,9 +34,9 @@
       <visual>
         <origin
-          xyz="0 0 0"
-          rpy="${-pi / 2} 0 0"/>
+          xyz="-0.125 -0.1 0.05"
+          rpy="${pi/2} 0 ${pi/2}"/>
         <geometry>
           <mesh
-            filename="package://kani_description/STL/base.stl"/>
+            filename="package://kani_description/meshes/base.stl"/>
         </geometry>
         <!-- <material>
@@ -46,9 +45,9 @@
       <collision>
         <origin
-          xyz="0 0 0"
+          xyz="-0.1 -0.125 0.06"
           rpy="0 0 0"/>
         <geometry>
           <mesh
-            filename="package://kani_description/STL/base.stl"/>
+            filename="package://kani_description/meshes/base.stl"/>
         </geometry>
         <!-- <material>

File: kani_description/urdf/wheels.urdf.xacro (robot description, xacro)
@@ -3,47 +3,49 @@
   <xacro:include filename="$(find kani_description)/urdf/base.transmission.xacro"/>
   <xacro:include filename="$(find kani_description)/urdf/base.gazebo.xacro" />
-  <xacro:property name="pi" value="3.1415926535897931" />
-  <xacro:property name="wheel_mesh" value="package://kani_description/STL/wheel_link.stl" />
-  <xacro:property name="steer_mesh" value="package://kani_description/STL/steer_link.stl" />
-  <xacro:macro name="wheel" params="parent x y z wheel_name">
-    <link name="${wheel_name}_wheel_link">
-      <inertial>
-        <origin
-          xyz="0 0 0"
-          rpy="0 0 0" /><!--0.00222524026865972 0.173009757872407 -0.000157420245397055-->
-        <mass
-          value="0.0963917377366023" />
-        <inertia
-          ixx="0.232225456967381"
-          ixy="0.0"
-          ixz="0.0"
-          iyy="0.232225456967381"
-          iyz="0.0"
-          izz="0.232225456967381" />
-      </inertial>
-      <visual>
-        <origin
-          xyz="0 0 0"
-          rpy="0 0 0" />
-        <geometry>
-          <mesh
-            filename="${wheel_mesh}" />
-        </geometry>
-        <material
-          name="black">
-        </material>
-      </visual>
-      <collision>
-        <origin
-          xyz="0 0 0"
-          rpy="0 0 0" />
-        <geometry>
-          <mesh
-            filename="${wheel_mesh}" />
-        </geometry>
-      </collision>
-    </link>
-    <joint
-      name="${wheel_name}_wheel_joint"
+  <xacro:property name="wheel_mesh" value="package://kani_description/meshes/wheel.stl" />
+  <xacro:property name="steer_mesh" value="package://kani_description/meshes/steer2.stl" />
+  <xacro:property name="steer_mesh_mirror" value="package://kani_description/meshes/steer2_m.stl" />
+  <!-- <xacro:property name="steer_eff" value="" />
+  <xacro:property name="steer_vel" value="" /> -->
+  <xacro:macro name="rf_wheel" params="parent x y z">
+    <link name="rightFront_wheel_link">
+      <inertial>
+        <origin
+          xyz="0 0 0"
+          rpy="0 0 0" /><!--0.00222524026865972 0.173009757872407 -0.000157420245397055-->
+        <mass
+          value="0.0963917377366023" />
+        <inertia
+          ixx="0.232225456967381"
+          ixy="0.0"
+          ixz="0.0"
+          iyy="0.232225456967381"
+          iyz="0.0"
+          izz="0.232225456967381" />
+      </inertial>
+      <visual>
+        <origin
+          xyz="${-0.1/3} 0 ${-0.1/3}"
+          rpy="${pi/2} 0 0" />
+        <geometry>
+          <mesh
+            filename="${wheel_mesh}" />
+        </geometry>
+        <material
+          name="black">
+        </material>
+      </visual>
+      <collision>
+        <origin
+          xyz="${-0.1/3} 0 ${-0.1/3}"
+          rpy="${pi/2} 0 0" />
+        <geometry>
+          <mesh
+            filename="${wheel_mesh}" />
+        </geometry>
+      </collision>
+    </link>
+    <joint
+      name="rightFront_wheel_joint"
       type="continuous">
       <origin
@@ -53,32 +55,32 @@
         link="${parent}" />
       <child
-        link="${wheel_name}_wheel_link" />
+        link="rightFront_wheel_link" />
       <axis
         xyz="0 1 0" />
     </joint>
     <!-- Extensions -->
-    <xacro:kani_wheel_gazebo link_name="${wheel_name}_wheel_link"/>
-    <xacro:kani_wheel_trans joint_name="${wheel_name}_wheel_joint"/>
-  </xacro:macro>
-  <xacro:macro name="steer" params="parent x y z steer_name">
-    <link name="${steer_name}_steer_link">
-      <inertial>
-        <origin
-          xyz="0 0 0"
-          rpy="0 0 0" /><!--0.00222524026865972 0.173009757872407 -0.000157420245397055-->
-        <mass
-          value="0.0963917377366023" />
-        <inertia
-          ixx="0.232225456967381"
-          ixy="0.0"
-          ixz="0.0"
-          iyy="0.232225456967381"
-          iyz="0.0"
-          izz="0.232225456967381" />
-      </inertial>
-      <visual>
-        <origin
-          xyz="0 0 0"
-          rpy="0 0 0" />
+    <xacro:kani_wheel_gazebo link_name="rightFront_wheel_link"/>
+    <xacro:kani_wheel_trans joint_name="rightFront_wheel_joint"/>
+  </xacro:macro>
+  <xacro:macro name="rf_steer" params="parent x y z">
+    <link name="rightFront_steer_link">
+      <inertial>
+        <origin
+          xyz="0 0 0"
+          rpy="${pi/2} 0 ${pi}" /><!--0.00222524026865972 0.173009757872407 -0.000157420245397055-->
+        <mass
+          value="0.0963917377366023" />
+        <inertia
+          ixx="0.232225456967381"
+          ixy="0.0"
+          ixz="0.0"
+          iyy="0.232225456967381"
+          iyz="0.0"
+          izz="0.232225456967381" />
+      </inertial>
+      <visual>
+        <origin
+          xyz="0.013 -0.01 0"
+          rpy="${pi/2} 0 ${pi}" />
         <geometry>
           <mesh
@@ -91,6 +93,6 @@
       <collision>
         <origin
-          xyz="0 0 0"
-          rpy="0 0 0" />
+          xyz="0.013 -0.01 0"
+          rpy="${pi/2} 0 ${pi}" />
         <geometry>
           <mesh
@@ -100,5 +102,66 @@
     </link>
     <joint
-      name="${steer_name}_steer_joint"
+      name="rightFront_steer_joint"
+      type="revolute">
+      <origin
+        xyz= "${x} ${y} ${z}"
+        rpy="0 0 0" /> <!-- xyz= "0.0600000000000003 -0.178955289353836 -0.0124450740677247" -->
+      <parent
+        link="${parent}" />
+      <child
+        link="rightFront_steer_link" />
+      <axis
+        xyz="0 0 1" />
+      <limit
+        lower="${-pi/2}"
+        upper="${pi/2}"
+        effort="500"
+        velocity="500"
+      />
+    </joint>
+    <!-- Extensions -->
+    <xacro:kani_steer_gazebo link_name="rightFront_steer_link"/>
+    <xacro:kani_steer_trans joint_name="rightFront_steer_joint"/>
+  </xacro:macro>
+  <xacro:macro name="rb_wheel" params="parent x y z">
+    <link name="rightBack_wheel_link">
+      <inertial>
+        <origin
+          xyz="0 0 0"
+          rpy="0 0 0" /><!--0.00222524026865972 0.173009757872407 -0.000157420245397055-->
+        <mass
+          value="0.0963917377366023" />
+        <inertia
+          ixx="0.232225456967381"
+          ixy="0.0"
+          ixz="0.0"
+          iyy="0.232225456967381"
+          iyz="0.0"
+          izz="0.232225456967381" />
+      </inertial>
+      <visual>
+        <origin
+          xyz="${-0.1/3} 0 ${-0.1/3}"
+          rpy="${pi/2} 0 0" />
+        <geometry>
+          <mesh
+            filename="${wheel_mesh}" />
+        </geometry>
+        <material
+          name="black">
+        </material>
+      </visual>
+      <collision>
+        <origin
+          xyz="${-0.1/3} 0 ${-0.1/3}"
+          rpy="${pi/2} 0 0" />
+        <geometry>
+          <mesh
+            filename="${wheel_mesh}" />
+        </geometry>
+      </collision>
+    </link>
+    <joint
+      name="rightBack_wheel_joint"
       type="continuous">
       <origin
@@ -108,11 +171,304 @@
         link="${parent}" />
       <child
-        link="${steer_name}_steer_link" />
+        link="rightBack_wheel_link" />
       <axis
         xyz="0 1 0" />
     </joint>
     <!-- Extensions -->
-    <xacro:kani_steer_gazebo link_name="${steer_name}_steer_link"/>
-    <xacro:kani_steer_trans joint_name="${steer_name}_steer_joint"/>
+    <xacro:kani_wheel_gazebo link_name="rightBack_wheel_link"/>
+    <xacro:kani_wheel_trans joint_name="rightBack_wheel_joint"/>
+  </xacro:macro>
+  <xacro:macro name="rb_steer" params="parent x y z">
+    <link name="rightBack_steer_link">
+      <inertial>
+        <origin
+          xyz="0 0 0"
+          rpy="${pi/2} 0 0" /><!--0.00222524026865972 0.173009757872407 -0.000157420245397055-->
+        <mass
+          value="0.0963917377366023" />
+        <inertia
+          ixx="0.232225456967381"
+          ixy="0.0"
+          ixz="0.0"
+          iyy="0.232225456967381"
+          iyz="0.0"
+          izz="0.232225456967381" />
+      </inertial>
+      <visual>
+        <origin
+          xyz="-0.013 0.047 0"
+          rpy="${pi/2} 0 0" />
+        <geometry>
+          <mesh
+            filename="${steer_mesh_mirror}" />
+        </geometry>
+        <material
+          name="black">
+        </material>
+      </visual>
+      <collision>
+        <origin
+          xyz="-0.013 0.047 0"
+          rpy="${pi/2} 0 0" />
+        <geometry>
+          <mesh
+            filename="${steer_mesh_mirror}" />
+        </geometry>
+      </collision>
+    </link>
+    <joint
+      name="rightBack_steer_joint"
+      type="revolute">
+      <origin
+        xyz= "${x} ${y} ${z}"
+        rpy="0 0 0" /> <!-- xyz= "0.0600000000000003 -0.178955289353836 -0.0124450740677247" -->
+      <parent
+        link="${parent}" />
+      <child
+        link="rightBack_steer_link" />
+      <axis
+        xyz="0 0 1" />
+      <limit
+        lower="${-pi/2}"
+        upper="${pi/2}"
+        effort="500"
+        velocity="500"
+      />
+    </joint>
+    <!-- Extensions -->
+    <xacro:kani_steer_gazebo link_name="rightBack_steer_link"/>
+    <xacro:kani_steer_trans joint_name="rightBack_steer_joint"/>
+  </xacro:macro>
+  <xacro:macro name="lf_wheel" params="parent x y z">
+    <link name="leftFront_wheel_link">
+      <inertial>
+        <origin
+          xyz="0 0 0"
+          rpy="0 0 0" /><!--0.00222524026865972 0.173009757872407 -0.000157420245397055-->
+        <mass
+          value="0.0963917377366023" />
+        <inertia
+          ixx="0.232225456967381"
+          ixy="0.0"
+          ixz="0.0"
+          iyy="0.232225456967381"
+          iyz="0.0"
+          izz="0.232225456967381" />
+      </inertial>
+      <visual>
+        <origin
+          xyz="${-0.1/3} 0 ${0.1/3}"
+          rpy="${-pi/2} 0 0" />
+        <geometry>
+          <mesh
+            filename="${wheel_mesh}" />
+        </geometry>
+        <material
+          name="black">
+        </material>
+      </visual>
+      <collision>
+        <origin
+          xyz="${-0.1/3} 0 ${0.1/3}"
+          rpy="${-pi/2} 0 0" />
+        <geometry>
+          <mesh
+            filename="${wheel_mesh}" />
+        </geometry>
+      </collision>
+    </link>
+    <joint
+      name="leftFront_wheel_joint"
+      type="continuous">
+      <origin
+        xyz= "${x} ${y} ${z}"
+        rpy="0 0 0" /> <!-- xyz= "0.0600000000000003 -0.178955289353836 -0.0124450740677247" -->
+      <parent
+        link="${parent}" />
+      <child
+        link="leftFront_wheel_link" />
+      <axis
+        xyz="0 1 0" />
+    </joint>
+    <!-- Extensions -->
+    <xacro:kani_wheel_gazebo link_name="leftFront_wheel_link"/>
+    <xacro:kani_wheel_trans joint_name="leftFront_wheel_joint"/>
+  </xacro:macro>
+  <xacro:macro name="lf_steer" params="parent x y z">
+    <link name="leftFront_steer_link">
+      <inertial>
+        <origin
+          xyz="0 0 0"
+          rpy="0 0 0" /><!--0.00222524026865972 0.173009757872407 -0.000157420245397055-->
+        <mass
+          value="0.0963917377366023" />
+        <inertia
+          ixx="0.232225456967381"
+          ixy="0.0"
+          ixz="0.0"
+          iyy="0.232225456967381"
+          iyz="0.0"
+          izz="0.232225456967381" />
+      </inertial>
+      <visual>
+        <origin
+          xyz="0.013 -0.047 0"
+          rpy="${pi/2} 0 ${pi}" />
+        <geometry>
+          <mesh
+            filename="${steer_mesh_mirror}" />
+        </geometry>
+        <material
+          name="black">
+        </material>
+      </visual>
+      <collision>
+        <origin
+          xyz="0.013 -0.047 0"
+          rpy="${pi/2} 0 ${pi}" />
+        <geometry>
+          <mesh
+            filename="${steer_mesh_mirror}" />
+        </geometry>
+      </collision>
+    </link>
+    <joint
+      name="leftFront_steer_joint"
+      type="revolute">
+      <origin
+        xyz= "${x} ${y} ${z}"
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