Commit message: update urdf model

File: kani_description/robots/kani.urdf.xacro (robot description, xacro)
@@ -1,4 +1,4 @@
 <?xml version="1.0"?>
-<robot name="kani" xmlns:xacro="http://www.ros.org/wiki/xacro">
+<robot name="kani" xmlns:xacro="http://ros.org/wiki/xacro">
   <xacro:property name="pi" value="3.1415926535897931" />
   <xacro:include filename="$(find kani_description)/urdf/base.urdf.xacro"/>
@@ -10,7 +10,7 @@
   <xacro:rb_steer parent="base_link" x="-0.092" y="-0.08875" z="-0.0039"/>
   <xacro:lb_steer parent="base_link" x="-0.092" y="0.08875" z="-0.0039" />
-  <xacro:rf_wheel parent="rightFront_steer_link" x="0" y="0" z="0"/>
-  <xacro:lf_wheel parent="leftFront_steer_link" x="0" y="0" z="0" />
-  <xacro:rb_wheel parent="rightBack_steer_link" x="0" y="0" z="0" />
-  <xacro:lb_wheel parent="leftBack_steer_link" x="0" y="0" z="0" />
+  <xacro:rf_wheel parent="rightFront_steer_link" x="0" y="0" z="-0.03945"/>
+  <xacro:lf_wheel parent="leftFront_steer_link" x="0" y="0" z="-0.03945" />
+  <xacro:rb_wheel parent="rightBack_steer_link" x="0" y="0" z="-0.03945" />
+  <xacro:lb_wheel parent="leftBack_steer_link" x="0" y="0" z="-0.03945" />
 </robot>

File: kani_description/urdf/base.transmission.xacro (robot description, xacro)
@@ -1,5 +1,5 @@
 <?xml version="1.0"?>
 <!-- Extensions -->
-<robot xmlns:xacro="http://www.ros.org/wiki/xacro">
+<robot xmlns:xacro="http://ros.org/wiki/xacro">
   <!-- wheel transmission -->
   <xacro:macro name="kani_wheel_trans" params="joint_name">

File: kani_description/urdf/base.urdf.xacro (robot description, xacro)
@@ -1,9 +1,9 @@
 <?xml version="1.0"?>
-<robot xmlns:xacro="http://www.ros.org/wiki/xacro">
+<robot xmlns:xacro="http://ros.org/wiki/xacro">
   <!-- <xacro:include filename="$(find kani_description)/urdf/base.transmission.xacro"/> -->
   <!-- <xacro:include filename="$(find kani_description)/urdf/base.gazebo.xacro" /> -->
   <xacro:include filename="$(find kani_description)/urdf/sensors/rplidar_A1.urdf.xacro" />
   <xacro:include filename="$(find kani_description)/urdf/sensors/_d435.urdf.xacro" />
-  <xacro:property name="base_height" value="0.06" />
+  <xacro:property name="base_height" value="0.05" />
   <xacro:macro name="kani_base">
     <link name="base_footprint">
@@ -37,9 +37,9 @@
       <visual>
         <origin
-          xyz="-0.125 -0.1 0"
-          rpy="${pi/2} 0 ${pi/2}"/>
+          xyz="-0.125 -0.1 -0"
+          rpy="0 0 0"/>
         <geometry>
           <mesh
-            filename="package://kani_description/meshes/base.stl"/>
+            filename="package://kani_description/meshes/base_v3.stl"/>
         </geometry>
         <!-- <material>
@@ -48,9 +48,9 @@
       <collision>
         <origin
-          xyz="-0.1 -0.125 0.06"
+          xyz="-0.125 -0.1 0"
           rpy="0 0 0"/>
         <geometry>
           <mesh
-            filename="package://kani_description/meshes/base.stl"/>
+            filename="package://kani_description/meshes/base_v3.stl"/>
         </geometry>
         <!-- <material>
@@ -58,18 +58,13 @@
       </collision>
     </link>
-    <!-- Wheel macros -->
-    <!-- <xacro:rwheel />
-    <xacro:lwheel /> -->
     <!-- intel realsense d435 utm30lx-->
     <sensor_d435 parent="base_link">
-      <origin xyz="0 0 -1" rpy="0 0 0"/>
+      <origin xyz="0.110 0.0 0.04" rpy="0 0 0"/>
     </sensor_d435>
     <sensor_a1 parent="base_link" name="laser">
-      <origin xyz="0 0 1" rpy="0 0 0"/>
+      <origin xyz="0.02 0.03 0.04" rpy="0 0 0"/>
     </sensor_a1>
-    <!-- <xacro:hokuyo_utm30lx name="hokuyo" parent="base_link"/> -->
-    <!-- <xacro:hokuyo_utm30lx_back name="hokuyo_back" parent="base_link"/> -->
     <!-- Extensions -->
-    <!-- <xacro:kani_base_gazebo/> -->
+    <xacro:kani_base_gazebo/>
   </xacro:macro>
 </robot>

File: kani_description/urdf/sensors/_d435.urdf.xacro (robot description, xacro)
@@ -7,4 +7,5 @@
 -->
 <robot name="sensor_d435" xmlns:xacro="http://ros.org/wiki/xacro">
+  <xacro:include filename="$(find kani_description)/urdf/sensors/_d435.gazebo.xacro" />
   <xacro:macro name="sensor_d435" params="parent *origin">
     <xacro:property name="M_PI" value="3.1415926535897931" />
@@ -63,4 +64,19 @@
         <inertia ixx="0.003881243" ixy="0.0" ixz="0.0" iyy="0.000498940" iyz="0.0" izz="0.003879257" />
       </inertial>
+      <sensor name="camera" type="depth">
+        <update_rate>20</update_rate>
+        <camera>
+          <horizontal_fov>1.047198</horizontal_fov>
+          <image>
+            <width>640</width>
+            <height>480</height>
+            <format>R8G8B8</format>
+          </image>
+          <clip>
+            <near>0.05</near>
+            <far>3</far>
+          </clip>
+        </camera>
+      </sensor>
     </link>
     <!-- camera depth joints and links -->
@@ -116,4 +132,7 @@
     </joint>
     <link name="camera_color_optical_frame"/>
+    <!-- assume the rgb camera on the depth lens frame -->
+    <!-- assume kinect as camera -->
+    <xacro:realsense_d435_depth name="camera_depth_optical"/>
   </xacro:macro>
 </robot>

File: kani_description/urdf/sensors/rplidar_A1.urdf.xacro (robot description, xacro)
@@ -14,5 +14,6 @@
     <link name="${name}_link">
       <visual>
-      <origin xyz="0 0 0" rpy="0 0 0"/>
+      <origin xyz=" -0.00714 0.00714 0" rpy="0 0 ${-pi/2}"/>
+      <!-- -0.00714 0.00714 0 -->
         <geometry>
           <mesh filename="package://kani_description/meshes/rplidar.stl"/>
@@ -21,5 +22,5 @@
       </visual>
       <collision>
-        <origin xyz="0 0 0" rpy="0 0 0"/>
+        <origin xyz="-0.00714 -0.00714 0" rpy="0 0 ${pi/2}"/>
         <geometry>
           <mesh filename="package://kani_description/meshes/rplidar.stl"/>

File: kani_description/urdf/wheels.urdf.xacro (robot description, xacro)
@@ -1,9 +1,9 @@
 <?xml version="1.0"?>
-<robot xmlns:xacro="http://www.ros.org/wiki/xacro">
+<robot xmlns:xacro="http://ros.org/wiki/xacro">
   <xacro:include filename="$(find kani_description)/urdf/base.transmission.xacro"/>
   <xacro:include filename="$(find kani_description)/urdf/base.gazebo.xacro" />
   <xacro:property name="wheel_mesh" value="package://kani_description/meshes/wheel.stl" />
-  <xacro:property name="steer_mesh" value="package://kani_description/meshes/steer2.stl" />
-  <xacro:property name="steer_mesh_mirror" value="package://kani_description/meshes/steer2_m.stl" />
+  <xacro:property name="steer_mesh" value="package://kani_description/meshes/steer_v3_meter_mirror.stl" />
+  <!-- <xacro:property name="steer_mesh" value="package://kani_description/meshes/steer_v3_meter_mirror.stl" /> -->
   <!-- <xacro:property name="steer_eff" value="" />
   <xacro:property name="steer_vel" value="" /> -->
@@ -26,5 +26,5 @@
       <visual>
         <origin
-          xyz="${-0.1/3} 0 ${-0.1/3}"
+          xyz="${-0.1/3} 0.009 ${-0.1/3}"
           rpy="${pi/2} 0 0" />
         <geometry>
@@ -38,5 +38,5 @@
       <collision>
         <origin
-          xyz="${-0.1/3} 0 ${-0.1/3}"
+          xyz="${-0.1/3} 0.009 ${-0.1/3}"
           rpy="${pi/2} 0 0" />
         <geometry>
@@ -68,31 +68,31 @@
         <origin
           xyz="0 0 0"
-          rpy="${pi/2} 0 ${pi}" /><!--0.00222524026865972 0.173009757872407 -0.000157420245397055-->
-        <mass
-          value="0.0963917377366023" />
-        <inertia
-          ixx="0.232225456967381"
-          ixy="0.0"
-          ixz="0.0"
-          iyy="0.232225456967381"
-          iyz="0.0"
-          izz="0.232225456967381" />
-      </inertial>
-      <visual>
-        <origin
-          xyz="0.013 -0.01 0"
-          rpy="${pi/2} 0 ${pi}" />
-        <geometry>
-          <mesh
-            filename="${steer_mesh}" />
-        </geometry>
-        <material
-          name="black">
-        </material>
-      </visual>
-      <collision>
-        <origin
-          xyz="0.013 -0.01 0"
-          rpy="${pi/2} 0 ${pi}" />
+          rpy="0 0 0" /><!--0.00222524026865972 0.173009757872407 -0.000157420245397055-->
+        <mass
+          value="0.0963917377366023" />
+        <inertia
+          ixx="0.232225456967381"
+          ixy="0.0"
+          ixz="0.0"
+          iyy="0.232225456967381"
+          iyz="0.0"
+          izz="0.232225456967381" />
+      </inertial>
+      <visual>
+        <origin
+          xyz="0.03875 0.0475 -0.059"
+          rpy="0 0 ${pi}" />
+        <geometry>
+          <mesh
+            filename="${steer_mesh}" />
+        </geometry>
+        <material
+          name="black">
+        </material>
+      </visual>
+      <collision>
+        <origin
+          xyz="0.03875 0.0475 -0.059"
+          rpy="0 0 ${pi}" />
         <geometry>
           <mesh
@@ -142,5 +142,5 @@
       <visual>
         <origin
-          xyz="${-0.1/3} 0 ${-0.1/3}"
+          xyz="${-0.1/3} 0.009 ${-0.1/3}"
           rpy="${pi/2} 0 0" />
         <geometry>
@@ -154,5 +154,5 @@
       <collision>
         <origin
-          xyz="${-0.1/3} 0 ${-0.1/3}"
+          xyz="${-0.1/3} 0.009 ${-0.1/3}"
           rpy="${pi/2} 0 0" />
         <geometry>
@@ -197,21 +197,21 @@
       <visual>
         <origin
-          xyz="-0.013 0.047 0"
-          rpy="${pi/2} 0 0" />
-        <geometry>
-          <mesh
-            filename="${steer_mesh_mirror}" />
-        </geometry>
-        <material
-          name="black">
-        </material>
-      </visual>
-      <collision>
-        <origin
-          xyz="-0.013 0.047 0"
-          rpy="${pi/2} 0 0" />
-        <geometry>
-          <mesh
-            filename="${steer_mesh_mirror}" />
+          xyz="0.03875 0.0475 -0.059"
+          rpy="0 0 ${pi}" />
+        <geometry>
+          <mesh
+            filename="${steer_mesh}" />
+        </geometry>
+        <material
+          name="black">
+        </material>
+      </visual>
+      <collision>
+        <origin
+          xyz="0.03875 0.0475 -0.059"
+          rpy="0 0 ${pi}" />
+        <geometry>
+          <mesh
+            filename="${steer_mesh}" />
         </geometry>
       </collision>
@@ -258,5 +258,5 @@
       <visual>
         <origin
-          xyz="${-0.1/3} 0 ${0.1/3}"
+          xyz="${-0.1/3} -0.009 ${0.1/3}"
           rpy="${-pi/2} 0 0" />
         <geometry>
@@ -270,5 +270,5 @@
       <collision>
         <origin
-          xyz="${-0.1/3} 0 ${0.1/3}"
+          xyz="${-0.1/3} -0.009 ${0.1/3}"
           rpy="${-pi/2} 0 0" />
         <geometry>
@@ -313,21 +313,21 @@
       <visual>
         <origin
-          xyz="0.013 -0.047 0"
-          rpy="${pi/2} 0 ${pi}" />
-        <geometry>
-          <mesh
-            filename="${steer_mesh_mirror}" />
-        </geometry>
-        <material
-          name="black">
-        </material>
-      </visual>
-      <collision>
-        <origin
-          xyz="0.013 -0.047 0"
-          rpy="${pi/2} 0 ${pi}" />
-        <geometry>
-          <mesh
-            filename="${steer_mesh_mirror}" />
+          xyz="-0.03875 -0.0475 -0.059"
+          rpy="0 0 0" />
+        <geometry>
+          <mesh
+            filename="${steer_mesh}" />
+        </geometry>
+        <material
+          name="black">
+        </material>
+      </visual>
+      <collision>
+        <origin
+          xyz="-0.03875 -0.0475 -0.059"
+          rpy="0 0 0" />
+        <geometry>
+          <mesh
+            filename="${steer_mesh}" />
         </geometry>
       </collision>
@@ -374,5 +374,5 @@
       <visual>
         <origin
-          xyz="${-0.1/3} 0 ${0.1/3}"
+          xyz="${-0.1/3} -0.009 ${0.1/3}"
           rpy="${-pi/2} 0 0" />
         <geometry>
@@ -386,5 +386,5 @@
       <collision>
         <origin
-          xyz="${-0.1/3} 0 ${0.1/3}"
+          xyz="${-0.1/3} -0.009 ${0.1/3}"
           rpy="${-pi/2} 0 0" />
         <geometry>
@@ -429,18 +429,18 @@
       <visual>
         <origin
-          xyz="-0.013 0.01 0"
-          rpy="${pi/2} 0 0" />
-        <geometry>
-          <mesh
-            filename="${steer_mesh}" />
-        </geometry>
-        <material
-          name="black">
-        </material>
-      </visual>
-      <collision>
-        <origin
-          xyz="-0.013 0.01 0"
-          rpy="${pi/2} 0 0" />
+          xyz="-0.03875 -0.0475 -0.059"
+          rpy="0 0 0" />
+        <geometry>
+          <mesh
+            filename="${steer_mesh}" />
+        </geometry>
+        <material
+          name="black">
+        </material>
+      </visual>
+      <collision>
+        <origin
+          xyz="-0.03875 -0.0475 -0.059"
+          rpy="0 0 0" />
         <geometry>
           <mesh
