Commit message: update inertia and mass and robot is able to move slowly

File: kani_description/robots/kani.urdf.xacro (robot description, xacro)
@@ -10,7 +10,7 @@
   <xacro:rb_steer parent="base_link" x="-0.092" y="-0.08875" z="-0.0039"/>
   <xacro:lb_steer parent="base_link" x="-0.092" y="0.08875" z="-0.0039" />
-  <xacro:rf_wheel parent="rightFront_steer_link" x="0" y="0" z="-0.03945"/>
-  <xacro:lf_wheel parent="leftFront_steer_link" x="0" y="0" z="-0.03945" />
-  <xacro:rb_wheel parent="rightBack_steer_link" x="0" y="0" z="-0.03945" />
-  <xacro:lb_wheel parent="leftBack_steer_link" x="0" y="0" z="-0.03945" />
+  <xacro:rf_wheel parent="rightFront_steer_link" x="0" y="0" z="-0.03395"/>
+  <xacro:lf_wheel parent="leftFront_steer_link" x="0" y="0" z="-0.03395" />
+  <xacro:rb_wheel parent="rightBack_steer_link" x="0" y="0" z="-0.03395" />
+  <xacro:lb_wheel parent="leftBack_steer_link" x="0" y="0" z="-0.03395" />
 </robot>

File: kani_description/urdf/base.gazebo.xacro (robot description, xacro)
@@ -12,10 +12,22 @@
     </gazebo>
   </xacro:macro>
+  <!-- steers -->
+  <xacro:macro name="kani_steer_gazebo" params="link_name">
+    <gazebo reference="${link_name}">
+      <material>Gazebo/Red</material>
+      <mu1 value="0.01"/>
+      <mu2 value="0.01"/>
+      <kp value="1000000.0" />
+      <kd value="1.0" />
+      <fdir1 value="1 0 0"/>
+      <dampingFactor value="0.00"/>
+    </gazebo>
+  </xacro:macro>
   <!-- wheels -->
   <xacro:macro name="kani_wheel_gazebo" params="link_name">
     <gazebo reference="${link_name}">
       <material>Gazebo/Black</material>
-      <mu1 value="100.0"/>
-      <mu2 value="100.0"/>
+      <mu1 value="0.2"/>
+      <mu2 value="0.2"/>
       <kp value="1000000.0"/>
       <kd value="1.0"/>
@@ -24,16 +36,3 @@
     </gazebo>
   </xacro:macro>
-  <xacro:macro name="kani_steer_gazebo" params="link_name">
-    <gazebo reference="${link_name}">
-      <material>Gazebo/Red</material>
-      <!-- fix below params?-->
-      <mu1 value="100.0"/>
-      <mu2 value="100.0"/>
-      <kp value="1000000.0" />
-      <kd value="1.0" />
-      <fdir1 value="1 0 0"/>
-      <dampingFactor value="0.1"/>
-      <!-- fix above params? -->
-    </gazebo>
-  </xacro:macro>
 </robot>

File: kani_description/urdf/base.urdf.xacro (robot description, xacro)
@@ -5,5 +5,5 @@
   <xacro:include filename="$(find kani_description)/urdf/sensors/rplidar_A1.urdf.xacro" />
   <xacro:include filename="$(find kani_description)/urdf/sensors/_d435.urdf.xacro" />
-  <xacro:property name="base_height" value="0.05" />
+  <xacro:property name="base_height" value="0.07" />
   <xacro:macro name="kani_base">
     <link name="base_footprint">
@@ -21,4 +21,5 @@
     </joint>
     <link name="base_link">
+      <gravity>1</gravity>
       <inertial>
         <origin
@@ -26,12 +27,12 @@
           rpy="0 0 0"/>
         <mass
-          value="0.05"/>
+          value="2"/>
         <inertia
-          ixx="0.2"
+          ixx="4e-3"
           ixy="0"
           ixz="0"
-          iyy="0.2"
+          iyy="3e-3"
           iyz="0"
-          izz="0.2"/>
+          izz="7e-3"/>
       </inertial>
       <visual>
@@ -60,8 +61,8 @@
     <!-- intel realsense d435 utm30lx-->
     <sensor_d435 parent="base_link">
-      <origin xyz="0.110 0.0 0.04" rpy="0 0 0"/>
+      <origin xyz="0.110 0.0 0.02" rpy="0 0 0"/>
     </sensor_d435>
     <sensor_a1 parent="base_link" name="laser">
-      <origin xyz="0.02 0.03 0.04" rpy="0 0 0"/>
+      <origin xyz="0.02 0.03 0.02" rpy="0 0 0"/>
     </sensor_a1>
     <!-- Extensions -->

File: kani_description/urdf/sensors/rplidar_A1.urdf.xacro (robot description, xacro)
@@ -22,5 +22,5 @@
       </visual>
       <collision>
-        <origin xyz="-0.00714 -0.00714 0" rpy="0 0 ${pi/2}"/>
+        <origin xyz="-0.00714 0.00714 0" rpy="0 0 ${-pi/2}"/>
         <geometry>
           <mesh filename="package://kani_description/meshes/rplidar.stl"/>

File: kani_description/urdf/wheels.urdf.xacro (robot description, xacro)
@@ -12,15 +12,15 @@
       <inertial>
         <origin
-          xyz="0 0 0"
-          rpy="0 0 0" /><!--0.00222524026865972 0.173009757872407 -0.000157420245397055-->
-        <mass
-          value="0.0963917377366023" />
-        <inertia
-          ixx="0.232225456967381"
-          ixy="0.0"
-          ixz="0.0"
-          iyy="0.232225456967381"
-          iyz="0.0"
-          izz="0.232225456967381" />
+          xyz="${-0.1/3} 0.009 ${-0.1/3}"
+          rpy="${pi/2} 0 0" /><!--0.00222524026865972 0.173009757872407 -0.000157420245397055-->
+        <mass
+          value="0.1" />
+        <inertia
+          ixx="1e-5"
+          ixy="0.0"
+          ixz="0.0"
+          iyy="1e-5"
+          iyz="0.0"
+          izz="1e-5" />
       </inertial>
       <visual>
@@ -67,19 +67,19 @@
       <inertial>
         <origin
-          xyz="0 0 0"
-          rpy="0 0 0" /><!--0.00222524026865972 0.173009757872407 -0.000157420245397055-->
-        <mass
-          value="0.0963917377366023" />
-        <inertia
-          ixx="0.232225456967381"
-          ixy="0.0"
-          ixz="0.0"
-          iyy="0.232225456967381"
-          iyz="0.0"
-          izz="0.232225456967381" />
-      </inertial>
-      <visual>
-        <origin
-          xyz="0.03875 0.0475 -0.059"
+          xyz="0.03875 0.0475 -0.0535"
+          rpy="0 0 ${pi}" /><!--0.00222524026865972 0.173009757872407 -0.000157420245397055-->
+        <mass
+          value="0.1" />
+        <inertia
+          ixx="6e-4"
+          ixy="0.0"
+          ixz="0.0"
+          iyy="6e-4"
+          iyz="0.0"
+          izz="6e-4" />
+      </inertial>
+      <visual>
+        <origin
+          xyz="0.03875 0.0475 -0.0535"
           rpy="0 0 ${pi}" />
         <geometry>
@@ -93,5 +93,5 @@
       <collision>
         <origin
-          xyz="0.03875 0.0475 -0.059"
+          xyz="0.03875 0.0475 -0.0535"
           rpy="0 0 ${pi}" />
         <geometry>
@@ -116,6 +116,6 @@
         lower="${-pi/2}"
         upper="${pi/2}"
-        effort="500"
-        velocity="500"
+        effort="80"
+        velocity="3"
       />
     </joint>
@@ -128,15 +128,15 @@
       <inertial>
         <origin
-          xyz="0 0 0"
-          rpy="0 0 0" /><!--0.00222524026865972 0.173009757872407 -0.000157420245397055-->
-        <mass
-          value="0.0963917377366023" />
-        <inertia
-          ixx="0.232225456967381"
-          ixy="0.0"
-          ixz="0.0"
-          iyy="0.232225456967381"
-          iyz="0.0"
-          izz="0.232225456967381" />
+          xyz="${-0.1/3} 0.009 ${-0.1/3}"
+          rpy="${pi/2} 0 0" /><!--0.00222524026865972 0.173009757872407 -0.000157420245397055-->
+        <mass
+          value="0.1" />
+        <inertia
+          ixx="1e-5"
+          ixy="0.0"
+          ixz="0.0"
+          iyy="1e-5"
+          iyz="0.0"
+          izz="1e-5" />
       </inertial>
       <visual>
@@ -183,19 +183,19 @@
       <inertial>
         <origin
-          xyz="0 0 0"
-          rpy="${pi/2} 0 0" /><!--0.00222524026865972 0.173009757872407 -0.000157420245397055-->
-        <mass
-          value="0.0963917377366023" />
-        <inertia
-          ixx="0.232225456967381"
-          ixy="0.0"
-          ixz="0.0"
-          iyy="0.232225456967381"
-          iyz="0.0"
-          izz="0.232225456967381" />
-      </inertial>
-      <visual>
-        <origin
-          xyz="0.03875 0.0475 -0.059"
+          xyz="0.03875 0.0475 -0.0535"
+          rpy="0 0 ${pi}" /><!--0.00222524026865972 0.173009757872407 -0.000157420245397055-->
+        <mass
+          value="0.1" />
+        <inertia
+          ixx="6e-4"
+          ixy="0.0"
+          ixz="0.0"
+          iyy="6e-4"
+          iyz="0.0"
+          izz="6e-4"/>
+      </inertial>
+      <visual>
+        <origin
+          xyz="0.03875 0.0475 -0.0535"
           rpy="0 0 ${pi}" />
         <geometry>
@@ -209,5 +209,5 @@
       <collision>
         <origin
-          xyz="0.03875 0.0475 -0.059"
+          xyz="0.03875 0.0475 -0.0535"
           rpy="0 0 ${pi}" />
         <geometry>
@@ -232,6 +232,6 @@
         lower="${-pi/2}"
         upper="${pi/2}"
-        effort="500"
-        velocity="500"
+        effort="80"
+        velocity="3"
       />
     </joint>
@@ -244,15 +244,15 @@
       <inertial>
         <origin
-          xyz="0 0 0"
-          rpy="0 0 0" /><!--0.00222524026865972 0.173009757872407 -0.000157420245397055-->
-        <mass
-          value="0.0963917377366023" />
-        <inertia
-          ixx="0.232225456967381"
-          ixy="0.0"
-          ixz="0.0"
-          iyy="0.232225456967381"
-          iyz="0.0"
-          izz="0.232225456967381" />
+          xyz="${-0.1/3} -0.009 ${0.1/3}"
+          rpy="${-pi/2} 0 0"  /><!--0.00222524026865972 0.173009757872407 -0.000157420245397055-->
+        <mass
+          value="0.1" />
+        <inertia
+          ixx="1e-5"
+          ixy="0.0"
+          ixz="0.0"
+          iyy="1e-5"
+          iyz="0.0"
+          izz="1e-5" />
       </inertial>
       <visual>
@@ -299,19 +299,19 @@
       <inertial>
         <origin
-          xyz="0 0 0"
-          rpy="0 0 0" /><!--0.00222524026865972 0.173009757872407 -0.000157420245397055-->
-        <mass
-          value="0.0963917377366023" />
-        <inertia
-          ixx="0.232225456967381"
-          ixy="0.0"
-          ixz="0.0"
-          iyy="0.232225456967381"
-          iyz="0.0"
-          izz="0.232225456967381" />
-      </inertial>
-      <visual>
-        <origin
-          xyz="-0.03875 -0.0475 -0.059"
+          xyz="-0.03875 -0.0475 -0.0535"
+          rpy="0 0 0"/><!--0.00222524026865972 0.173009757872407 -0.000157420245397055-->
+        <mass
+          value="0.1" />
+        <inertia
+          ixx="6e-4"
+          ixy="0.0"
+          ixz="0.0"
+          iyy="6e-4"
+          iyz="0.0"
+          izz="6e-4"/>
+      </inertial>
+      <visual>
+        <origin
+          xyz="-0.03875 -0.0475 -0.0535"
           rpy="0 0 0" />
         <geometry>
@@ -325,5 +325,5 @@
       <collision>
         <origin
-          xyz="-0.03875 -0.0475 -0.059"
+          xyz="-0.03875 -0.0475 -0.0535"
           rpy="0 0 0" />
         <geometry>
@@ -348,6 +348,6 @@
         lower="${-pi/2}"
         upper="${pi/2}"
-        effort="500"
-        velocity="500"
+        effort="80"
+        velocity="3"
       />
     </joint>
@@ -360,15 +360,15 @@
       <inertial>
         <origin
-          xyz="0 0 0"
-          rpy="0 0 0" /><!--0.00222524026865972 0.173009757872407 -0.000157420245397055-->
-        <mass
-          value="0.0963917377366023" />
-        <inertia
-          ixx="0.232225456967381"
-          ixy="0.0"
-          ixz="0.0"
-          iyy="0.232225456967381"
-          iyz="0.0"
-          izz="0.232225456967381" />
+          xyz="${-0.1/3} -0.009 ${0.1/3}"
+          rpy="${-pi/2} 0 0" /><!--0.00222524026865972 0.173009757872407 -0.000157420245397055-->
+        <mass
+          value="0.1" />
+        <inertia
+          ixx="1e-5"
+          ixy="0.0"
+          ixz="0.0"
+          iyy="1e-5"
+          iyz="0.0"
+          izz="1e-5" />
       </inertial>
       <visual>
@@ -415,19 +415,19 @@
       <inertial>
         <origin
-          xyz="0 0 0"
+          xyz="-0.03875 -0.0475 -0.0535"
           rpy="0 0 0" /><!--0.00222524026865972 0.173009757872407 -0.000157420245397055-->
         <mass
-          value="0.0963917377366023" />
-        <inertia
-          ixx="0.232225456967381"
-          ixy="0.0"
-          ixz="0.0"
-          iyy="0.232225456967381"
-          iyz="0.0"
-          izz="0.232225456967381" />
-      </inertial>
-      <visual>
-        <origin
-          xyz="-0.03875 -0.0475 -0.059"
+          value="0.1" />
+        <inertia
+          ixx="6e-4"
+          ixy="0.0"
+          ixz="0.0"
+          iyy="6e-4"
+          iyz="0.0"
+          izz="6e-4"/>
+      </inertial>
+      <visual>
+        <origin
+          xyz="-0.03875 -0.0475 -0.0535"
           rpy="0 0 0" />
         <geometry>
@@ -441,5 +441,5 @@
       <collision>
         <origin
-          xyz="-0.03875 -0.0475 -0.059"
+          xyz="-0.03875 -0.0475 -0.0535"
           rpy="0 0 0" />
         <geometry>
@@ -464,6 +464,6 @@
         lower="${-pi/2}"
         upper="${pi/2}"
-        effort="500"
-        velocity="500"
+        effort="80"
+        velocity="3"
       />
     </joint>
